Commit message: feat: implement true inverse kinematics in MotorController and update URDF dimensions for improved accuracy

File: ambers_ws/src/phoenix_description/urdf/phoenix.urdf (robot description, URDF)
Before this commit: robot phoenix, 8 links, 7 joints
Links:
- link base_link: mass 5.0 -> 5.4; geometry collision box size=0.465 0.355 0.200; visual box size=0.465 0.355 0.200
- link front_left_wheel: geometry collision cylinder length=0.026 radius=0.0325; visual cylinder length=0.026 radius=0.0325
- link front_right_wheel: geometry collision cylinder length=0.026 radius=0.0325; visual cylinder length=0.026 radius=0.0325
- link rear_left_wheel: geometry collision cylinder length=0.026 radius=0.0325; visual cylinder length=0.026 radius=0.0325
- link rear_right_wheel: geometry collision cylinder length=0.026 radius=0.0325; visual cylinder length=0.026 radius=0.0325
Joints:
- joint camera_joint: origin xyz=0.27 0 0.125 rpy=0 0 0 -> xyz=0.2325 0 0.100 rpy=0 0 0
- joint front_left_wheel_joint: origin xyz=0.2 0.175 0 rpy=-1.5708 0 0 -> xyz=0.200 0.175 0 rpy=-1.5708 0 0
- joint front_right_wheel_joint: origin xyz=0.2 -0.175 0 rpy=-1.5708 0 0 -> xyz=0.200 -0.175 0 rpy=-1.5708 0 0
- joint lidar_joint: origin xyz=0 0 0.26 rpy=0 0 0 -> xyz=0 0 0.21 rpy=0 0 0
- joint rear_left_wheel_joint: origin xyz=-0.2 0.175 0 rpy=-1.5708 0 0 -> xyz=-0.200 0.175 0 rpy=-1.5708 0 0
- joint rear_right_wheel_joint: origin xyz=-0.2 -0.175 0 rpy=-1.5708 0 0 -> xyz=-0.200 -0.175 0 rpy=-1.5708 0 0

Commit message: fix: update maximum linear speed and adjust wheel dimensions in URDF for improved performance

File: ambers_ws/src/phoenix_description/urdf/phoenix.urdf (robot description, URDF)
Before this commit: robot phoenix, 8 links, 7 joints
Links:
- added link nozzle_link, mass 0.1; collision cylinder length=0.08 radius=0.012; visual cylinder length=0.08 radius=0.012
- added link pan_link, mass 0.1; collision cylinder length=0.04 radius=0.030; visual cylinder length=0.04 radius=0.030
- link camera_link: geometry collision box size=0.025 0.024 0.015; visual box size=0.025 0.024 0.015
- link front_left_wheel: geometry collision cylinder length=0.05 radius=0.065; visual cylinder length=0.05 radius=0.065
- link front_right_wheel: geometry collision cylinder length=0.05 radius=0.065; visual cylinder length=0.05 radius=0.065
- link rear_left_wheel: geometry collision cylinder length=0.05 radius=0.065; visual cylinder length=0.05 radius=0.065
- link rear_right_wheel: geometry collision cylinder length=0.05 radius=0.065; visual cylinder length=0.05 radius=0.065
Joints:
- added joint pan_joint: type continuous, parent base_link, child pan_link, origin xyz=0.210 0 0.200 rpy=0 0 0, axis 0 0 1
- added joint tilt_joint: type revolute, parent pan_link, child nozzle_link, origin xyz=0.020 0 0.050 rpy=0 0 0, axis 0 1 0, limit lower=-0.7854 upper=0.7854 effort=10.0 velocity=3.0
- joint camera_joint: origin xyz=0.2325 0 0.100 rpy=0 0 0 -> xyz=0.035 0 -0.022 rpy=0 0 0; parent base_link -> nozzle_link
- joint lidar_joint: origin xyz=0 0 0.21 rpy=0 0 0 -> xyz=-0.120 0 0.210 rpy=0 0 0

Commit message: upgrades

File: ambers_ws/src/phoenix_description/urdf/phoenix.urdf (robot description, URDF)
Before this commit: robot phoenix, 10 links, 9 joints
Joints:
- joint lidar_joint: origin xyz=-0.120 0 0.210 rpy=0 0 0 -> xyz=0.100 0 0.300 rpy=0 0 0
